File: hardware/pcb/pcb.kicad_sch (KiCad schematic)
At the start: 30 parts, among them J1 L_GPIO, J2 R_GPIO, J3 USB_C_Receptacle_USB2.0_14P, U1 ESP32-C3-WROOM-02, U3 TPS62291

Commit message: add neeko
Parts:
- D-RX1, D-RXOK1, D-SFD1, D-TX1, DWM1, R6, R7, R8, R9: now not fitted
- R10, R11: LCSC Part C413002 -> C2791532
Changed lines of the file:
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@@
 		(in_bom yes)
 		(on_board yes)
-		(dnp no)
+		(dnp yes)
 		(property "Reference" "D-RXOK1"
 			(at 217.17 109.22 0)
@@
 		(in_bom yes)
 		(on_board yes)
-		(dnp no)
+		(dnp yes)
 		(property "Reference" "D-TX1"
 			(at 217.17 135.89 0)
@@
 		(in_bom yes)
 		(on_board yes)
-		(dnp no)
+		(dnp yes)
 		(property "Reference" "D-RX1"
 			(at 217.17 127 0)
@@
 		(in_bom yes)
 		(on_board yes)
-		(dnp no)
+		(dnp yes)
 		(property "Reference" "D-SFD1"
 			(at 217.17 118.11 0)
@@
 		(in_bom yes)
 		(on_board yes)
-		(dnp no)
+		(dnp yes)
 		(fields_autoplaced yes)
 		(property "Reference" "R9"
@@
 		(in_bom yes)
 		(on_board yes)
-		(dnp no)
+		(dnp yes)
 		(fields_autoplaced yes)
 		(property "Reference" "R6"
@@
 			)
 		)
-		(property "LCSC Part" "C413002"
+		(property "LCSC Part" "C2791532"
 			(at 50.8 147.32 90)
 			(effects
@@
 			)
 		)
-		(property "LCSC Part" "C413002"
+		(property "LCSC Part" "C2791532"
 			(at 50.8 149.86 90)
 			(effects
@@
 		(in_bom yes)
 		(on_board yes)
-		(dnp no)
+		(dnp yes)
 		(fields_autoplaced yes)
 		(property "Reference" "DWM1"
@@
 		(in_bom yes)
 		(on_board yes)
-		(dnp no)
+		(dnp yes)
 		(fields_autoplaced yes)
 		(property "Reference" "R8"
@@
 		(in_bom yes)
 		(on_board yes)
-		(dnp no)
+		(dnp yes)
 		(fields_autoplaced yes)
 		(property "Reference" "R7"

Commit message: reroute dálnice for backlit lightbulb
Parts:
- added D1: LED, LED_SMD:LED_0201_0603Metric_Pad0.64x0.40mm_HandSolder, symbol Device:LED
- added R12: R, Resistor_SMD:R_0402_1005Metric, symbol Device:R
- D-RX1, D-RXOK1, D-SFD1, D-TX1: footprint LED_SMD:LED_0402_1005Metric -> LED_SMD:LED_0402_1005Metric_Pad0.77x0.64mm_HandSolder
- R6, R7, R8, R9: footprint Resistor_SMD:R_0402_1005Metric -> Resistor_SMD:R_0402_1005Metric_Pad0.72x0.64mm_HandSolder
Connections:
- net +3V3: now also R12.2
- net GND: now also D1.1 (K)
- new net: D1.2 (A), R12.1
